File: Hardware/Magnetic-Imaging-Tile.sch (EAGLE design)
At the start: 90 parts, among them U01 DRV5053, U02 DRV5053, U03 DRV5053, U04 DRV5053, U05 DRV5053, U06 DRV5053, U07 DRV5053, U08 CD74HC4067, U09 DRV5053, U10 DRV5053, U104 SN74HC590A, U105 SN74LVC1G139, U106 AD7680, U11 DRV5053, U12 DRV5053, U13 DRV5053, U14 DRV5053, U15 DRV5053, U16 DRV5053, U17 DRV5053, U18 CD74HC4067, U19 CD74HC4067, U20 DRV5053, U21 DRV5053, U22 DRV5053, U23 DRV5053, U24 DRV5053, U25 DRV5053, U26 DRV5053, U27 DRV5053, U28 CD74HC4067, U30 DRV5053, U31 DRV5053, U32 DRV5053, U33 DRV5053, U34 DRV5053, U35 DRV5053, U36 DRV5053, U37 DRV5053, U40 DRV5053, U41 DRV5053, U42 DRV5053, U43 DRV5053, U44 DRV5053, U45 DRV5053, U46 DRV5053, U47 DRV5053, U50 DRV5053, U51 DRV5053, U52 DRV5053, U53 DRV5053, U54 DRV5053, U55 DRV5053, U56 DRV5053, U57 DRV5053, U60 DRV5053, U61 DRV5053, U62 DRV5053, U63 DRV5053, U64 DRV5053, U65 DRV5053, U66 DRV5053, U67 DRV5053, U70 DRV5053, U71 DRV5053, U72 DRV5053, U73 DRV5053, U74 DRV5053, U75 DRV5053, U76 DRV5053, U77 DRV5053

Commit message: Update
-Changes silk to vector
-Added order instructions
-Updated Design By
-OSH and SPARKFUN added to sch and board as part
Parts:
- added LOGO1: SPECIAL_INSTRUCTIONS-ORDERING, SparkFun-Aesthetics:SPECIAL_INSTRUCTIONS-ORDERING
- added LOGO3: SFE_LOGO_NAME.1_INCH, SparkFun-Aesthetics:SFE_LOGO_NAME.1_INCH
- added LOGO4: OSHW-LOGOS, SparkFun-Aesthetics:OSHW-LOGOS
Other:
- note added: "Peter Jansen Revised by: Chris Bryant"
- note added: "V10"
Changed lines of the file:
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@@
 <layer number="56" name="wert" color="7" fill="1" visible="no" active="no"/>
 <layer number="57" name="tCAD" color="7" fill="1" visible="no" active="no"/>
+<layer number="58" name="bCopper" color="7" fill="1" visible="no" active="no"/>
 <layer number="59" name="tCarbon" color="7" fill="1" visible="no" active="no"/>
 <layer number="60" name="bCarbon" color="7" fill="1" visible="no" active="no"/>
@@
 <layer number="128" name="_bValues" color="7" fill="1" visible="yes" active="yes"/>
 <layer number="129" name="Mask" color="7" fill="1" visible="yes" active="yes"/>
+<layer number="130" name="SMDSTROOK" color="7" fill="1" visible="no" active="no"/>
 <layer number="131" name="tAdjust" color="7" fill="1" visible="yes" active="yes"/>
 <layer number="132" name="bAdjust" color="7" fill="1" visible="yes" active="yes"/>
+<layer number="133" name="bottom_silk" color="7" fill="1" visible="no" active="no"/>
+<layer number="134" name="silk_top" color="7" fill="1" visible="no" active="no"/>
+<layer number="135" name="silk_bottom" color="7" fill="1" visible="no" active="no"/>
+<layer number="136" name="silktop" color="7" fill="1" visible="no" active="no"/>
+<layer number="137" name="silkbottom" color="7" fill="1" visible="no" active="no"/>
+<layer number="138" name="EEE" color="7" fill="1" visible="no" active="no"/>
+<layer number="139" name="_tKeepout" color="7" fill="1" visible="no" active="no"/>
+<layer number="140" name="mbKeepout" color="7" fill="1" visible="no" active="no"/>
+<layer number="141" name="ASSEMBLY_TOP" color="7" fill="1" visible="no" active="no"/>
+<layer number="142" name="mbRestrict" color="7" fill="1" visible="no" active="no"/>
+<layer number="143" name="PLACE_BOUND_TOP" color="7" fill="1" visible="no" active="no"/>
 <layer number="144" name="Drill_legend" color="7" fill="1" visible="no" active="yes"/>
+<layer number="145" name="DrillLegend_01-16" color="7" fill="1" visible="no" active="no"/>
+<layer number="146" name="DrillLegend_01-20" color="7" fill="1" visible="no" active="no"/>
+<layer number="147" name="PIN_NUMBER" color="7" fill="1" visible="no" active="no"/>
+<layer number="148" name="DrillLegend_01-20" color="7" fill="1" visible="no" active="no"/>
+<layer number="149" name="DrillLegend_02-15" color="7" fill="1" visible="no" active="no"/>
 <layer number="150" name="Notes" color="7" fill="1" visible="yes" active="yes"/>
 <layer number="151" name="HeatSink" color="7" fill="1" visible="no" active="yes"/>
@@
 <layer number="154" name="FabDoc2" color="7" fill="1" visible="yes" active="yes"/>
 <layer number="155" name="FabDoc3" color="7" fill="1" visible="yes" active="yes"/>
+<layer number="156" name="gesam-Maß" color="1" fill="7" visible="no" active="no"/>
+<layer number="157" name="FaceMchng" color="3" fill="1" visible="no" active="no"/>
+<layer number="158" name="FaceMMeas" color="3" fill="1" visible="no" active="no"/>
+<layer number="159" name="Geh-Bear2" color="1" fill="7" visible="no" active="no"/>
+<layer number="160" name="Topologie" color="9" fill="1" visible="no" active="no"/>
+<layer number="161" name="tomplace2" color="7" fill="1" visible="no" active="no"/>
+<layer number="166" name="AntennaArea" color="7" fill="1" visible="no" active="no"/>
+<layer number="168" name="4mmHeightArea" color="7" fill="1" visible="no" active="no"/>
+<layer number="191" name="mNets" color="7" fill="1" visible="no" active="no"/>
+<layer number="192" name="mBusses" color="7" fill="1" visible="no" active="no"/>
+<layer number="193" name="mPins" color="7" fill="1" visible="no" active="no"/>
+<layer number="194" name="mSymbols" color="7" fill="1" visible="no" active="no"/>
+<layer number="195" name="mNames" color="7" fill="1" visible="no" active="no"/>
+<layer number="196" name="mValues" color="7" fill="1" visible="no" active="no"/>
 <layer number="199" name="Contour" color="7" fill="1" visible="yes" active="yes"/>
 <layer number="200" name="200bmp" color="1" fill="10" visible="no" active="yes"/>
@@
 <layer number="250" name="Descript" color="3" fill="1" visible="no" active="no"/>
 <layer number="251" name="SMDround" color="12" fill="11" visible="no" active="no"/>
+<layer number="252" name="BR-BS" color="7" fill="1" visible="no" active="no"/>
+<layer number="253" name="Extra" color="7" fill="1" visible="no" active="no"/>
 <layer number="254" name="cooling" color="7" fill="1" visible="no" active="yes"/>
 <layer number="255" name="routoute" color="7" fill="1" visible="yes" active="yes"/>
@@
 <part name="U19" library="SparkFun-IC-Logic" deviceset="74*4067" device="SM96" technology="HC" value="CD74HC4067"/>
 <part name="U28" library="SparkFun-IC-Logic" deviceset="74*4067" device="SM96" technology="HC" value="CD74HC4067"/>
+<part name="LOGO3" library="SparkFun-Aesthetics" deviceset="SFE_LOGO_NAME" device=".1_INCH"/>
+<part name="LOGO4" library="SparkFun-Aesthetics" deviceset="OSHW-LOGO" device="S"/>
+<part name="LOGO1" library="SparkFun-Aesthetics" deviceset="SPECIAL_INSTRUCTIONS" device="-ORDERING"/>
 </parts>
 <sheets>
@@
 <plain>
 <text x="17.78" y="66.04" size="1.778" layer="97">The sensor used is the DRV5053VA: -90mV/mT sensitivity</text>
+<text x="350.52" y="7.62" size="2.54" layer="94" font="vector">Peter Jansen
+Revised by: Chris Bryant</text>
+<text x="421.64" y="7.62" size="1.778" layer="94" font="vector">V10</text>
 </plain>
 <instances>
@@
 <attribute name="VALUE" x="165.1" y="99.06" size="1.778" layer="95" font="vector" rot="MR0"/>
 </instance>
+<instance part="LOGO3" gate="G$1" x="335.28" y="33.02" smashed="yes"/>
+<instance part="LOGO4" gate="G$1" x="406.4" y="45.72" smashed="yes"/>
+<instance part="LOGO1" gate="G$1" x="408.94" y="20.32" smashed="yes"/>
 </instances>
 <busses>
@@
 </schematic>
 </drawing>
+<compatibility>
+<note version="6.3" minversion="6.2.2" severity="warning">
+Since Version 6.2.2 text objects can contain more than one line,
+which will not be processed correctly with this version.
+</note>
+</compatibility>
 </eagle>
